Commit message: Updates

File: eagleye_util/tf/urdf/sensors.xacro (robot description, xacro)
@@ -3,5 +3,5 @@
   xmlns:xacro="http://ros.org/wiki/xacro">
   <xacro:arg name="config_dir" default="$(find eagleye_tf)"/>
-  <xacro:property name="calibration" value="${xacro.load_yaml,('$(arg config_dir)/config/sensors_tf.yaml')}"/>
+  <xacro:property name="calibration" value="${xacro.load_yaml('$(arg config_dir)/config/sensors_tf.yaml')}"/>
   <xacro:property name="size" value="1" />
   <!-- base_link -->
